File: KiCad/AutoWater/AutoWater.kicad_sch (KiCad schematic)
At the start: 46 parts, among them IC1 74ABT125PW, P1 Pump, SW1 Button, SW2 Button, Y1 32.768 kHz

Commit message: Refactoring schema
Parts:
- BT1: footprint (none) -> AutoWater:Connector 5.5x2.1 DS-201
- BT2: footprint (none) -> AutoWater:Batary box CR2032
- C1, C4: footprint (none) -> AutoWater:Capacitor Murata SMD 0402
- C2, C3: footprint (none) -> AutoWater:Capacitor Murata SMD 0603
- D1: value ~ -> 1N4001G; footprint (none) -> AutoWater:DIode 1N4001G THT min
- D2: value ~ -> green; footprint (none) -> AutoWater:LED 3mm
- D3, D4, D7: value ~ -> red; footprint (none) -> AutoWater:LED 3mm
- D5, D6, D8: value ~ -> yellow; footprint (none) -> AutoWater:LED 3mm
- D9: value ~ -> orange; footprint (none) -> AutoWater:LED 3mm
- LCD1: footprint (none) -> AutoWater:PLS-4
- MCU1: footprint (none) -> AutoWater:Arduino Nano V3 Type C PBS
- P1: footprint (none) -> AutoWater:Connector B2B-XH-A
- Q1: value ~ -> BC817-25; footprint (none) -> AutoWater:NPN transistor BC817-25
- R1: footprint (none) -> AutoWater:Resistor Rohm SMD 0603
- R10, R11, R12, R13, R14, R15, R16, R17, R6, R7, R8, R9: footprint (none) -> AutoWater:Resistor Yageo SMD 1206
- R2, R3, R4, R5: footprint (none) -> AutoWater:Resistor Yageo SMD 0805
- REG1: footprint (none) -> AutoWater:Register 74HC164M SOP-14
- RTC1: footprint (none) -> AutoWater:RTC DS1307 DIP
- RV1, RV2: footprint (none) -> AutoWater:PLS-3
- SD1: footprint (none) -> AutoWater:MicroSD
- STB1: footprint (none) -> AutoWater:Stabilizer 5V AMS1117-5.0S SMD
- SW1, SW2: footprint (none) -> AutoWater:PLS-2
- Y1: footprint (none) -> AutoWater:Crystal 32768 SMD
