File: KiCad/AutoWater/state_module.kicad_sch (KiCad schematic)
At the start: 18 parts

Commit message: Create layouts
Parts:
- D2, D3, D4, D5, D6, D7, D8, D9: renamed from D?; footprint (none) -> AutoWater:LED 3mm
- R10, R11, R4, R5, R6, R7, R8, R9: renamed from R?; footprint (none) -> AutoWater:Resistor Yageo SMD 1206
- REG1: renamed from REG?; footprint (none) -> AutoWater:Register 74HC164M SOP-14
- SM2: renamed from SM?; footprint (none) -> AutoWater:PLS-4
Connections:
- net at REG1.CLK: now also SM2.3 (CLK); no longer SM2.CLK
- net at REG1.DSA, REG1.Rst, REG1.Vin: now also SM2.1 (Vin); no longer SM2.Vin
- net at REG1.DSB: now also SM2.2 (SER); no longer SM2.SER
- net at D2.GND, D3.GND, D4.GND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: now also SM2.4 (GND); no longer SM2.GND
Other:
- moved on the sheet: SM2
Changed lines of the file:
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@@
+	(wire
+		(pts
+			(xy 24.13 52.07) (xy 24.13 63.5)
+		)
+		(stroke
+			(width 0)
+			(type default)
+		)
+	)
 	(wire
 		(pts
@@
 		(pts
 			(xy 34.29 21.59) (xy 24.13 21.59)
-		)
-		(stroke
-			(width 0)
-			(type default)
-		)
-	)
-	(wire
-		(pts
-			(xy 24.13 49.53) (xy 24.13 63.5)
 		)
 		(stroke
@@
 		(dnp no)
 		(fields_autoplaced yes)
-		(property "Reference" "REG?"
+		(property "Reference" "REG1"
 			(at 45.72 46.99 0)
 			(do_not_autoplace yes)
@@
 			)
 		)
-		(property "Footprint" ""
+		(property "Footprint" "AutoWater:Register 74HC164M SOP-14"
 			(at 39.37 26.67 0)
 			(effects
@@
 			(project ""
 				(path "/9c9c7373-5af3-48f7-b840-36e6b46427ae/60800294-856f-4bcb-a194-133197c72ad2"
-					(reference "REG?")
+					(reference "REG1")
 					(unit 1)
 				)
@@
 		(dnp no)
 		(fields_autoplaced yes)
-		(property "Reference" "R?"
+		(property "Reference" "R4"
 			(at 71.12 20.32 0)
 			(do_not_autoplace yes)
@@
 			)
 		)
-		(property "Footprint" ""
+		(property "Footprint" "AutoWater:Resistor Yageo SMD 1206"
 			(at 69.342 22.86 90)
 			(effects
@@
 			(project ""
 				(path "/9c9c7373-5af3-48f7-b840-36e6b46427ae/60800294-856f-4bcb-a194-133197c72ad2"
-					(reference "R?")
+					(reference "R4")
 					(unit 1)
 				)
@@
 		(dnp no)
 		(fields_autoplaced yes)
-		(property "Reference" "D?"
+		(property "Reference" "D6"
 			(at 81.28 40.64 0)
 			(do_not_autoplace yes)
@@
 			)
 		)
-		(property "Footprint" ""
+		(property "Footprint" "AutoWater:LED 3mm"
 			(at 81.28 43.18 0)
 			(effects
@@
 			(project ""
 				(path "/9c9c7373-5af3-48f7-b840-36e6b46427ae/60800294-856f-4bcb-a194-133197c72ad2"
-					(reference "D?")
+					(reference "D6")
 					(unit 1)
 				)
@@
 		(dnp no)
 		(fields_autoplaced yes)
-		(property "Reference" "D?"
+		(property "Reference" "D9"
 			(at 81.28 55.88 0)
 			(do_not_autoplace yes)
@@
 			)
 		)
-		(property "Footprint" ""
+		(property "Footprint" "AutoWater:LED 3mm"
 			(at 81.28 58.42 0)
 			(effects
@@
 			(project ""
 				(path "/9c9c7373-5af3-48f7-b840-36e6b46427ae/60800294-856f-4bcb-a194-133197c72ad2"
-					(reference "D?")
+					(reference "D9")
 					(unit 1)
 				)
@@
 		(dnp no)
 		(fields_autoplaced yes)
-		(property "Reference" "R?"
+		(property "Reference" "R8"
 			(at 71.12 40.64 0)
 			(do_not_autoplace yes)
@@
 			)
 		)
-		(property "Footprint" ""
+		(property "Footprint" "AutoWater:Resistor Yageo SMD 1206"
 			(at 69.342 43.18 90)
 			(effects
@@
 			(project ""
 				(path "/9c9c7373-5af3-48f7-b840-36e6b46427ae/60800294-856f-4bcb-a194-133197c72ad2"
-					(reference "R?")
+					(reference "R8")
 					(unit 1)
 				)
@@
 		(dnp no)
 		(fields_autoplaced yes)
-		(property "Reference" "D?"
+		(property "Reference" "D4"
 			(at 81.28 30.48 0)
 			(do_not_autoplace yes)
@@
 			)
 		)
-		(property "Footprint" ""
+		(property "Footprint" "AutoWater:LED 3mm"
 			(at 81.28 33.02 0)
 			(effects
@@
 			(project ""
 				(path "/9c9c7373-5af3-48f7-b840-36e6b46427ae/60800294-856f-4bcb-a194-133197c72ad2"
-					(reference "D?")
+					(reference "D4")
 					(unit 1)
 				)
@@
 		(dnp no)
 		(fields_autoplaced yes)
-		(property "Reference" "SM?"
-			(at 24.13 36.83 0)
+		(property "Reference" "SM2"
+			(at 21.59 41.91 0)
 			(do_not_autoplace yes)
 			(effects
@@
 			)
 		)
-		(property "Footprint" ""
+		(property "Footprint" "AutoWater:PLS-4"
 			(at 19.05 34.29 0)
 			(effects
@@
 			)
 		)
-		(pin "SER"
-		)
-		(pin "CLK"
-		)
-		(pin "GND"
-		)
-		(pin "Vin"
-		)
-		(instances
-			(project ""
-				(path "/9c9c7373-5af3-48f7-b840-36e6b46427ae/60800294-856f-4bcb-a194-133197c72ad2"
-					(reference "SM?")
+		(pin "2"
+		)
+		(pin "1"
+		)
+		(pin "4"
+		)
+		(pin "3"
+		)
+		(instances
+			(project ""
+				(path "/9c9c7373-5af3-48f7-b840-36e6b46427ae/60800294-856f-4bcb-a194-133197c72ad2"
+					(reference "SM2")
 					(unit 1)
 				)
@@
 		(dnp no)
 		(fields_autoplaced yes)
-		(property "Reference" "R?"
+		(property "Reference" "R6"
 			(at 71.12 30.48 0)
 			(do_not_autoplace yes)
@@
 			)
 		)
-		(property "Footprint" ""
+		(property "Footprint" "AutoWater:Resistor Yageo SMD 1206"
 			(at 69.342 33.02 90)
 			(effects
@@
 			(project ""
 				(path "/9c9c7373-5af3-48f7-b840-36e6b46427ae/60800294-856f-4bcb-a194-133197c72ad2"
-					(reference "R?")
+					(reference "R6")
 					(unit 1)
 				)
@@
 		(dnp no)
 		(fields_autoplaced yes)
-		(property "Reference" "R?"
+		(property "Reference" "R10"
 			(at 71.12 50.8 0)
 			(do_not_autoplace yes)
@@
 			)
 		)
-		(property "Footprint" ""
+		(property "Footprint" "AutoWater:Resistor Yageo SMD 1206"
 			(at 69.342 53.34 90)
 			(effects
@@
 			(project ""
 				(path "/9c9c7373-5af3-48f7-b840-36e6b46427ae/60800294-856f-4bcb-a194-133197c72ad2"
-					(reference "R?")
+					(reference "R10")
 					(unit 1)
 				)
@@
 		(dnp no)
 		(fields_autoplaced yes)
-		(property "Reference" "R?"
+		(property "Reference" "R5"
 			(at 71.12 25.4 0)
 			(do_not_autoplace yes)
@@
 			)
 		)
-		(property "Footprint" ""
+		(property "Footprint" "AutoWater:Resistor Yageo SMD 1206"
 			(at 69.342 27.94 90)
 			(effects
@@
 			(project ""
 				(path "/9c9c7373-5af3-48f7-b840-36e6b46427ae/60800294-856f-4bcb-a194-133197c72ad2"
-					(reference "R?")
+					(reference "R5")
 					(unit 1)
 				)
@@
 		(dnp no)
 		(fields_autoplaced yes)
-		(property "Reference" "R?"
+		(property "Reference" "R9"
 			(at 71.12 45.72 0)
 			(do_not_autoplace yes)
@@
 			)
 		)
-		(property "Footprint" ""
+		(property "Footprint" "AutoWater:Resistor Yageo SMD 1206"
 			(at 69.342 48.26 90)
 			(effects
@@
 			(project ""
 				(path "/9c9c7373-5af3-48f7-b840-36e6b46427ae/60800294-856f-4bcb-a194-133197c72ad2"
-					(reference "R?")
+					(reference "R9")
 					(unit 1)
 				)
@@
 		(dnp no)
 		(fields_autoplaced yes)
-		(property "Reference" "R?"
+		(property "Reference" "R11"
 			(at 71.12 55.88 0)
 			(do_not_autoplace yes)
@@
 			)
 		)
-		(property "Footprint" ""
+		(property "Footprint" "AutoWater:Resistor Yageo SMD 1206"
 			(at 69.342 58.42 90)
 			(effects
@@
 			(project ""
 				(path "/9c9c7373-5af3-48f7-b840-36e6b46427ae/60800294-856f-4bcb-a194-133197c72ad2"
-					(reference "R?")
+					(reference "R11")
 					(unit 1)
 				)
@@
 		(dnp no)
 		(fields_autoplaced yes)
-		(property "Reference" "D?"
+		(property "Reference" "D8"
 			(at 81.28 50.8 0)
 			(do_not_autoplace yes)
@@
 			)
 		)
-		(property "Footprint" ""
+		(property "Footprint" "AutoWater:LED 3mm"
 			(at 81.28 53.34 0)
 			(effects
@@
 			(project ""
 				(path "/9c9c7373-5af3-48f7-b840-36e6b46427ae/60800294-856f-4bcb-a194-133197c72ad2"
-					(reference "D?")
+					(reference "D8")
 					(unit 1)
 				)
@@
 		(dnp no)
 		(fields_autoplaced yes)
-		(property "Reference" "D?"
+		(property "Reference" "D7"
 			(at 81.28 45.72 0)
 			(do_not_autoplace yes)
@@
 			)
 		)
-		(property "Footprint" ""
+		(property "Footprint" "AutoWater:LED 3mm"
 			(at 81.28 48.26 0)
 			(effects
@@
 			(project ""
 				(path "/9c9c7373-5af3-48f7-b840-36e6b46427ae/60800294-856f-4bcb-a194-133197c72ad2"
-					(reference "D?")
+					(reference "D7")
 					(unit 1)
 				)
@@
 		(dnp no)
 		(fields_autoplaced yes)
-		(property "Reference" "D?"
+		(property "Reference" "D3"
 			(at 81.28 25.4 0)
 			(do_not_autoplace yes)
@@
 			)
 		)
-		(property "Footprint" ""
+		(property "Footprint" "AutoWater:LED 3mm"
 			(at 81.28 27.94 0)
 			(effects
@@
 			(project ""
 				(path "/9c9c7373-5af3-48f7-b840-36e6b46427ae/60800294-856f-4bcb-a194-133197c72ad2"
-					(reference "D?")
+					(reference "D3")
 					(unit 1)
 				)
@@
 		(dnp no)
 		(fields_autoplaced yes)
-		(property "Reference" "D?"
+		(property "Reference" "D5"
 			(at 81.28 35.56 0)
 			(do_not_autoplace yes)
@@
 			)
 		)
-		(property "Footprint" ""
+		(property "Footprint" "AutoWater:LED 3mm"
 			(at 81.28 38.1 0)
 			(effects
@@
 			(project ""
 				(path "/9c9c7373-5af3-48f7-b840-36e6b46427ae/60800294-856f-4bcb-a194-133197c72ad2"
-					(reference "D?")
+					(reference "D5")
 					(unit 1)
 				)
@@
 		(dnp no)
 		(fields_autoplaced yes)
-		(property "Reference" "R?"
+		(property "Reference" "R7"
 			(at 71.12 35.56 0)
 			(do_not_autoplace yes)
@@
 			)
 		)
-		(property "Footprint" ""
+		(property "Footprint" "AutoWater:Resistor Yageo SMD 1206"
 			(at 69.342 38.1 90)
 			(effects
@@
 			(project ""
 				(path "/9c9c7373-5af3-48f7-b840-36e6b46427ae/60800294-856f-4bcb-a194-133197c72ad2"
-					(reference "R?")
+					(reference "R7")
 					(unit 1)
 				)
@@
 		(dnp no)
 		(fields_autoplaced yes)
-		(property "Reference" "D?"
+		(property "Reference" "D2"
 			(at 81.28 20.32 0)
 			(do_not_autoplace yes)
@@
 			)
 		)
-		(property "Footprint" ""
+		(property "Footprint" "AutoWater:LED 3mm"
 			(at 81.28 22.86 0)
 			(effects
@@
 			(project ""
 				(path "/9c9c7373-5af3-48f7-b840-36e6b46427ae/60800294-856f-4bcb-a194-133197c72ad2"
-					(reference "D?")
-					(unit 1)
-				)
+					(reference "D2")
+					(unit 1)
+				)
