File: KiCad/AutoWater/water_module.kicad_sch (KiCad schematic)
At the start: 8 parts

Commit message: Create layouts
Parts:
- C3: renamed from C?; footprint (none) -> AutoWater:Capacitor Murata SMD 0402
- D1: renamed from D?; footprint (none) -> AutoWater:DIode 1N4001G THT min
- P1: renamed from P?; footprint (none) -> AutoWater:Connector B2B-XH-A
- Q1: renamed from Q?; footprint (none) -> AutoWater:NPN transistor BC817-25
- R3: renamed from R?; footprint (none) -> AutoWater:Resistor Yageo SMD 1206
- RV1, RV2: renamed from RV?; footprint (none) -> AutoWater:PLS-3
- WM2: renamed from WM?; footprint (none) -> AutoWater:PLS-2x3
Other:
- moved on the sheet: C3, D1, P1, Q1, R3, RV1, RV2, WM2
